File: floppyv3_expansion.kicad_pcb (KiCad board)
At the start: 2 copper layers, 69 x 69 mm, 20 parts, among them J1 Left_Bank_Free_Socket, J2 Left_Bank_Board_Socket, J3 STLink_Board_Conn, J4 Right_Bank_Board_Socket, J5 Right_Bank_Free_Socket, J6 FTSH-107-01-L-DV-K-TR, SW1 USR_BTN, U1 MAX6816

Commit message: Updated to production version
Parts:
- moved C1 1.00 mm to (115.2, 116.6)
- moved U1 0.59 mm to (115.1, 120.9)
Routing:
- net Net-(U1-IN): track 18.3 -> 14.2 mm
- net /3V3: track 135.3 -> 135.9 mm
- net GND: vias 28 -> 29
Changed lines of the file:
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@@
 	(footprint "Package_TO_SOT_SMD:SOT-143"
 		(layer "B.Cu")
-		(at 115.13 120.31 180)
+		(at 115.1 120.9 180)
 		(descr "SOT-143 https://www.nxp.com/docs/en/package-information/SOT143B.pdf")
 		(tags "SOT-143")
 		(property "Reference" "U1"
-			(at 0.02 4.11 0)
+			(at 0.03 -2.45 0)
 			(layer "B.SilkS")
 			(effects
@@
 	(footprint "Capacitor_SMD:C_0805_2012Metric"
 		(layer "B.Cu")
-		(at 115.15 117.6)
+		(at 115.15 116.6)
 		(descr "Capacitor SMD 0805 (2012 Metric), square (rectangular) end terminal, IPC-7351 nominal, (Body size source: IPC-SM-782 page 76, https://www.pcb-3d.com/wordpress/wp-content/uploads/ipc-sm-782a_amendment_1_and_2.pdf, https://docs.google.com/spreadsheets/d/1BsfQQcO9C6DZCsRaXUlFlo91Tg2WpOkGARC1WS5S8t0/edit?usp=sharing), generated with kicad-footprint-generator")
 		(tags "capacitor")
 		(property "Reference" "C1"
-			(at 0 5 0)
+			(at 0 -1.6 0)
 			(layer "B.SilkS")
 			(effects
@@
 	)
 	(via
+		(at 100.9 69.6)
+		(size 0.6)
+		(drill 0.3)
+		(layers "F.Cu" "B.Cu")
+		(free yes)
+		(net 1)
+	)
+	(via
 		(at 98.6 124)
 		(size 0.6)
@@
 	)
 	(segment
+		(start 109.2 111.6)
+		(end 114.2 116.6)
+		(width 0.4)
+		(layer "B.Cu")
+		(net 2)
+	)
+	(segment
+		(start 109.2 109.4)
+		(end 109.2 111.6)
+		(width 0.4)
+		(layer "B.Cu")
+		(net 2)
+	)
+	(segment
 		(start 109.2 107.2)
 		(end 109.2 109.4)
@@
 	)
 	(segment
-		(start 114.13 117.67)
-		(end 114.2 117.6)
-		(width 0.4)
-		(layer "B.Cu")
-		(net 2)
-	)
-	(segment
 		(start 112.56 85.56)
 		(end 112.56 87.145)
@@
 	)
 	(segment
-		(start 114.13 119.36)
-		(end 114.13 117.67)
-		(width 0.4)
-		(layer "B.Cu")
-		(net 2)
-	)
-	(segment
 		(start 109.2 82.2)
 		(end 112.56 85.56)
@@
 	)
 	(segment
+		(start 114.1 116.7)
+		(end 114.2 116.6)
+		(width 0.4)
+		(layer "B.Cu")
+		(net 2)
+	)
+	(segment
 		(start 109.2 79.4)
 		(end 109.2 82.2)
@@
 	)
 	(segment
-		(start 109.2 112.628014)
-		(end 114.18 117.608014)
-		(width 0.4)
-		(layer "B.Cu")
-		(net 2)
-	)
-	(segment
 		(start 93.71 118.94)
 		(end 91.8 118.94)
@@
 	)
 	(segment
+		(start 114.1 119.95)
+		(end 114.1 116.7)
+		(width 0.4)
+		(layer "B.Cu")
+		(net 2)
+	)
+	(segment
 		(start 93.71 118.94)
 		(end 95.25 117.4)
@@
 	)
 	(segment
-		(start 109.2 109.4)
-		(end 109.2 112.628014)
-		(width 0.4)
-		(layer "B.Cu")
-		(net 2)
-	)
-	(segment
 		(start 97.489 119.419)
 		(end 95.219 119.419)
@@
 	)
 	(segment
-		(start 112.67 119.8)
+		(start 114.1 121.85)
+		(end 112.05 119.8)
+		(width 0.2)
+		(layer "B.Cu")
+		(net 37)
+	)
+	(segment
+		(start 112.05 119.8)
 		(end 104.8 119.8)
 		(width 0.2)
@@
 	)
 	(segment
-		(start 114.13 121.26)
-		(end 112.67 119.8)
-		(width 0.2)
-		(layer "B.Cu")
-		(net 37)
-	)
-	(segment
-		(start 109.5035 121.861)
-		(end 120.8015 121.861)
+		(start 116.1 121.85)
+		(end 116.1 122.151)
 		(width 0.2)
 		(layer "B.Cu")
@@
 	)
 	(segment
-		(start 116.13 121.26)
+		(start 120.2115 122.451)
 		(end 121.4025 121.26)
 		(width 0.2)
@@
 	)
 	(segment
+		(start 116.1 122.151)
+		(end 115.8 122.451)
+		(width 0.2)
+		(layer "B.Cu")
+		(net 38)
+	)
+	(segment
 		(start 108.9025 121.26)
-		(end 109.5035 121.861)
+		(end 110.0935 122.451)
 		(width 0.2)
 		(layer "B.Cu")
@@
 	)
 	(segment
-		(start 120.8015 121.861)
-		(end 121.4025 121.26)
-		(width 0.2)
-		(layer "B.Cu")
+		(start 110.0935 122.451)
+		(end 115.8 122.451)
+		(width 0.2)
+		(layer "B.Cu")
+		(net 38)
+	)
+	(segment
+		(start 115.8 122.451)
+		(end 120.2115 122.451)
+		(width 0.2)
+		(layer "B.Cu")
